Commit message: Renamed package to be able to have the meshes

File: open_manipulator_support_description/urdf/open_manipulator_support.urdf.xacro (robot description, xacro)
@@ -3,11 +3,11 @@
 <robot name="open_manipulator" xmlns:xacro="http://www.ros.org/wiki/xacro">
 <!-- Import all Gazebo-customization elements, including Gazebo colors -->
-  <xacro:include filename="$(find open_manipulator_support)/urdf/open_manipulator.gazebo.xacro"/>
+  <xacro:include filename="$(find open_manipulator_support_description)/urdf/open_manipulator.gazebo.xacro"/>
 <!-- Import Rviz colors -->
-  <xacro:include filename="$(find open_manipulator_support)/urdf/materials.xacro" />
+  <xacro:include filename="$(find open_manipulator_support_description)/urdf/materials.xacro" />
 <!-- Import inertial Properties-->
-  <xacro:include filename="$(find open_manipulator_support)/urdf/inertial_properties.xacro" />
+  <xacro:include filename="$(find open_manipulator_support_description)/urdf/inertial_properties.xacro" />
 <!-- Import inertial Properties-->
-  <xacro:include filename="$(find open_manipulator_support)/urdf/mass_properties.xacro" />
+  <xacro:include filename="$(find open_manipulator_support_description)/urdf/mass_properties.xacro" />
  <!-- World -->
    <link name="world">
@@ -33,5 +33,5 @@
 	<visual>
 		<geometry>
-        	<mesh filename="package://open_manipulator_support/meshes/base_link.STL"/>
+        	<mesh filename="package://open_manipulator_support_description/meshes/base_link.STL"/>
 		</geometry>
 		<material name="grey"/>
@@ -39,5 +39,5 @@
 	<collision>
       <geometry>
-        <mesh filename="package://open_manipulator_support/meshes/base_link.STL" />
+        <mesh filename="package://open_manipulator_support_description/meshes/base_link.STL" />
       </geometry>
     </collision>
@@ -47,5 +47,5 @@
     <visual>
       <geometry>
-        <mesh filename="package://open_manipulator_support/meshes/link1.STL"/>
+        <mesh filename="package://open_manipulator_support_description/meshes/link1.STL"/>
       </geometry>
       <material name="grey"/>
@@ -53,5 +53,5 @@
     <collision>
       <geometry>
-        <mesh filename="package://open_manipulator_support/meshes/link1.STL"/>
+        <mesh filename="package://open_manipulator_support_description/meshes/link1.STL"/>
       </geometry>
     </collision>
@@ -91,5 +91,5 @@
 	<visual>
       <geometry>
-        <mesh filename="package://open_manipulator_support/meshes/link2.STL"/>
+        <mesh filename="package://open_manipulator_support_description/meshes/link2.STL"/>
       </geometry>
       <material name="grey"/>
@@ -97,5 +97,5 @@
     <collision>
       <geometry>
-        <mesh filename="package://open_manipulator_support/meshes/link2.STL"/>
+        <mesh filename="package://open_manipulator_support_description/meshes/link2.STL"/>
       </geometry>
     </collision>
@@ -135,5 +135,5 @@
     <visual>
       <geometry>
-        <mesh filename="package://open_manipulator_support/meshes/link3.STL"/>
+        <mesh filename="package://open_manipulator_support_description/meshes/link3.STL"/>
       </geometry>
       <material name="grey"/>
@@ -141,5 +141,5 @@
     <collision>
       <geometry>
-        <mesh filename="package://open_manipulator_support/meshes/link3.STL"/>
+        <mesh filename="package://open_manipulator_support_description/meshes/link3.STL"/>
       </geometry>
     </collision>
@@ -179,5 +179,5 @@
     <visual>
       <geometry>
-        <mesh filename="package://open_manipulator_support/meshes/link4.STL"/>
+        <mesh filename="package://open_manipulator_support_description/meshes/link4.STL"/>
       </geometry>
       <material name="grey"/>
@@ -185,5 +185,5 @@
     <collision>
       <geometry>
-        <mesh filename="package://open_manipulator_support/meshes/link4.STL"/>
+        <mesh filename="package://open_manipulator_support_description/meshes/link4.STL"/>
       </geometry>
     </collision>
@@ -223,5 +223,5 @@
     <visual>
       <geometry>
-        <mesh filename="package://open_manipulator_support/meshes/link5.STL"/>
+        <mesh filename="package://open_manipulator_support_description/meshes/link5.STL"/>
       </geometry>
       <material name="grey"/>
@@ -229,5 +229,5 @@
     <collision>
       <geometry>
-        <mesh filename="package://open_manipulator_support/meshes/link5.STL"/>
+        <mesh filename="package://open_manipulator_support_description/meshes/link5.STL"/>
       </geometry>
     </collision>
@@ -278,5 +278,5 @@
     <visual>
       <geometry>
-        <mesh filename="package://open_manipulator_support/meshes/link6.STL" />
+        <mesh filename="package://open_manipulator_support_description/meshes/link6.STL" />
       </geometry>
       <material name="grey" />
@@ -284,5 +284,5 @@
     <collision>
       <geometry>
-        <mesh filename="package://open_manipulator_support/meshes/link6.STL" />
+        <mesh filename="package://open_manipulator_support_description/meshes/link6.STL" />
       </geometry>
     </collision>
@@ -323,5 +323,5 @@
       <geometry>
         <mesh
-          filename="package://open_manipulator_support/meshes/link7.STL" />
+          filename="package://open_manipulator_support_description/meshes/link7.STL" />
       </geometry>
       <material name="grey" />
@@ -330,5 +330,5 @@
       <geometry>
         <mesh
-          filename="package://open_manipulator_support/meshes/link7.STL" />
+          filename="package://open_manipulator_support_description/meshes/link7.STL" />
       </geometry>
     </collision>
@@ -371,5 +371,5 @@
       <geometry>
         <mesh
-          filename="package://open_manipulator_support/meshes/gripper.STL" />
+          filename="package://open_manipulator_support_description/meshes/gripper.STL" />
       </geometry>
       <material name="grey" />
@@ -378,5 +378,5 @@
       <geometry>
         <mesh
-          filename="package://open_manipulator_support/meshes/gripper.STL" />
+          filename="package://open_manipulator_support_description/meshes/gripper.STL" />
       </geometry>
     </collision>
@@ -406,5 +406,5 @@
         <visual>
       <geometry>
-        <mesh filename="package://open_manipulator_support/meshes/gripper.STL" />
+        <mesh filename="package://open_manipulator_support_description/meshes/gripper.STL" />
       </geometry>
       <material name="grey" />
@@ -412,5 +412,5 @@
     <collision>
       <geometry>
-        <mesh filename="package://open_manipulator_support/meshes/gripper.STL" />
+        <mesh filename="package://open_manipulator_support_description/meshes/gripper.STL" />
       </geometry>
     </collision>
